File: 1_MAIN/1_Main.brd (EAGLE design)
At the start: 67.4 x 54.8 mm, 43 parts, among them IC1 NCP1117-33ST, IC10 FT232RL, IC2 MCP1700T-1802E, IC7 MAX14932, IC8 MAX14932, IC9 MAX14932, Q1 IRF7416, X14 ALLSERIALMM, X2 MINI-USB-32005-201, X3 AKL18X-04W

Commit message: Add BOM
Routing:
- net +12V/1: track 53.4 -> 55.2 mm, vias 0 -> 1
- net +3V3/1: track 75.6 -> 76.6 mm
- net +5V/1: track 59.4 -> 58.6 mm
Changed lines of the file:
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@@
 </element>
 <element name="C1" library="rcl" package="C0805" value="10n" x="-26.9875" y="11.43" smashed="yes" rot="R180">
-<attribute name="NAME" x="-27.305" y="10.4775" size="1.016" layer="25" rot="R180"/>
-<attribute name="VALUE" x="-26.3525" y="14.605" size="1.016" layer="27" rot="R180"/>
+<attribute name="NAME" x="-26.9875" y="10.4775" size="1.016" layer="25" rot="R180"/>
+<attribute name="VALUE" x="-25.7175" y="14.9225" size="1.016" layer="27" rot="R180"/>
 </element>
 <element name="C2" library="rcl" package="C0805" value="100n" x="-20.32" y="39.37" smashed="yes" rot="R180">
@@
 <contactref element="R3" pad="1"/>
 <contactref element="LED2" pad="C"/>
-<wire x1="10.91" y1="9.525" x2="12.065" y2="9.525" width="0.3048" layer="1"/>
-<wire x1="12.065" y1="9.525" x2="12.7" y2="10.16" width="0.3048" layer="1"/>
-<wire x1="12.7" y1="10.16" x2="14.925" y2="10.16" width="0.3048" layer="1"/>
+<wire x1="10.91" y1="9.525" x2="12.7" y2="9.525" width="0.3048" layer="1"/>
+<wire x1="12.7" y1="9.525" x2="13.335" y2="10.16" width="0.3048" layer="1"/>
+<wire x1="13.335" y1="10.16" x2="14.925" y2="10.16" width="0.3048" layer="1"/>
 </signal>
 <signal name="N$7">
@@
 <wire x1="-5.56" y1="11.275" x2="-8.255" y2="13.97" width="0.4064" layer="16"/>
 <wire x1="-8.255" y1="13.97" x2="-8.255" y2="22.225" width="0.4064" layer="16"/>
-<wire x1="-8.255" y1="22.225" x2="-15.875" y2="29.845" width="0.4064" layer="16"/>
-<wire x1="-15.875" y1="29.845" x2="-15.875" y2="43.18" width="0.4064" layer="16"/>
-<wire x1="-11.43" y1="45.085" x2="-13.97" y2="45.085" width="0.4064" layer="16"/>
-<wire x1="-15.875" y1="43.18" x2="-13.97" y2="45.085" width="0.4064" layer="16"/>
-<wire x1="-13.97" y1="45.085" x2="-15.875" y2="45.085" width="0.4064" layer="16"/>
-<wire x1="-15.875" y1="45.085" x2="-19.05" y2="48.26" width="0.4064" layer="16"/>
-<wire x1="-19.05" y1="48.26" x2="-19.05" y2="49.53" width="0.4064" layer="16"/>
+<wire x1="-8.255" y1="22.225" x2="-17.145" y2="31.115" width="0.4064" layer="16"/>
+<wire x1="-17.145" y1="31.115" x2="-17.145" y2="41.91" width="0.4064" layer="16"/>
+<via x="-17.145" y="41.91" extent="1-16" drill="0.3"/>
+<wire x1="-19.05" y1="49.53" x2="-19.05" y2="46.0375" width="0.4064" layer="1"/>
+<wire x1="-19.05" y1="46.0375" x2="-17.145" y2="44.1325" width="0.4064" layer="1"/>
+<wire x1="-17.145" y1="44.1325" x2="-17.145" y2="41.91" width="0.4064" layer="1"/>
+<wire x1="-11.43" y1="45.085" x2="-12.065" y2="45.085" width="0.4064" layer="1"/>
+<wire x1="-12.065" y1="45.085" x2="-13.97" y2="43.18" width="0.4064" layer="1"/>
+<wire x1="-13.97" y1="43.18" x2="-15.875" y2="43.18" width="0.4064" layer="1"/>
+<wire x1="-15.875" y1="43.18" x2="-17.145" y2="41.91" width="0.4064" layer="1"/>
 </signal>
 <signal name="+5V/1">
@@
 <wire x1="-2.06" y1="10.95" x2="-7.3025" y2="16.1925" width="0.4064" layer="16"/>
 <wire x1="-7.3025" y1="16.1925" x2="-7.3025" y2="22.5425" width="0.4064" layer="16"/>
-<wire x1="-7.3025" y1="22.5425" x2="-14.605" y2="29.845" width="0.4064" layer="16"/>
+<wire x1="-7.3025" y1="22.5425" x2="-15.875" y2="31.115" width="0.4064" layer="16"/>
 <wire x1="-8.89" y1="45.085" x2="-9.525" y2="45.085" width="0.4064" layer="1"/>
 <wire x1="-9.525" y1="45.085" x2="-10.16" y2="44.45" width="0.4064" layer="1"/>
 <wire x1="-10.16" y1="44.45" x2="-10.16" y2="41.91" width="0.4064" layer="1"/>
 <wire x1="-10.16" y1="41.91" x2="-12.7" y2="39.37" width="0.4064" layer="1"/>
-<wire x1="-14.605" y1="29.845" x2="-14.605" y2="34.29" width="0.4064" layer="16"/>
-<via x="-14.605" y="34.29" extent="1-16" drill="0.3"/>
+<wire x1="-15.875" y1="31.115" x2="-15.875" y2="34.29" width="0.4064" layer="16"/>
+<via x="-15.875" y="34.29" extent="1-16" drill="0.3"/>
 <wire x1="-17.8562" y1="34.0614" x2="-17.6276" y2="34.29" width="0.4064" layer="1"/>
-<wire x1="-17.6276" y1="34.29" x2="-14.605" y2="34.29" width="0.4064" layer="1"/>
+<wire x1="-17.6276" y1="34.29" x2="-15.875" y2="34.29" width="0.4064" layer="1"/>
 <wire x1="-19.37" y1="39.37" x2="-19.37" y2="36.83" width="0.4064" layer="1"/>
 <wire x1="-17.6276" y1="34.29" x2="-17.78" y2="34.29" width="0.4064" layer="1"/>
@@
 <wire x1="1.44" y1="9.355" x2="-6.35" y2="17.145" width="0.4064" layer="16"/>
 <wire x1="-6.35" y1="17.145" x2="-6.35" y2="22.86" width="0.4064" layer="16"/>
-<wire x1="-6.35" y1="22.86" x2="-13.6525" y2="30.1625" width="0.4064" layer="16"/>
+<wire x1="-6.35" y1="22.86" x2="-14.605" y2="31.115" width="0.4064" layer="16"/>
 <wire x1="-17.8562" y1="31.75" x2="-15.56" y2="31.75" width="0.4064" layer="1"/>
 <wire x1="-15.56" y1="31.75" x2="-15.24" y2="31.43" width="0.4064" layer="1"/>
@@
 <wire x1="-7.62" y1="41.91" x2="-11.1125" y2="38.4175" width="0.4064" layer="1"/>
 <wire x1="-11.1125" y1="38.4175" x2="-13.0175" y2="38.4175" width="0.4064" layer="1"/>
-<wire x1="-13.0175" y1="38.4175" x2="-13.6525" y2="37.7825" width="0.4064" layer="1"/>
-<wire x1="-13.6525" y1="37.7825" x2="-13.6525" y2="33.02" width="0.4064" layer="1"/>
-<via x="-13.6525" y="33.02" extent="1-16" drill="0.3"/>
-<wire x1="-13.6525" y1="30.1625" x2="-13.6525" y2="33.02" width="0.4064" layer="16"/>
-<wire x1="-15.24" y1="31.43" x2="-13.9725" y2="31.43" width="0.4064" layer="1"/>
-<wire x1="-13.9725" y1="31.43" x2="-13.6525" y2="31.75" width="0.4064" layer="1"/>
-<wire x1="-13.6525" y1="31.75" x2="-13.6525" y2="33.02" width="0.4064" layer="1"/>
 <wire x1="-24.054" y1="31.75" x2="-17.8562" y2="31.75" width="0.6096" layer="1"/>
+<wire x1="-14.605" y1="31.115" x2="-14.605" y2="34.29" width="0.4064" layer="16"/>
+<via x="-14.605" y="34.29" extent="1-16" drill="0.3"/>
+<wire x1="-13.0175" y1="38.4175" x2="-14.605" y2="36.83" width="0.4064" layer="1"/>
+<wire x1="-14.605" y1="36.83" x2="-14.605" y2="34.29" width="0.4064" layer="1"/>
+<wire x1="-15.24" y1="31.43" x2="-15.24" y2="33.02" width="0.4064" layer="1"/>
+<wire x1="-15.24" y1="33.02" x2="-14.605" y2="33.655" width="0.4064" layer="1"/>
+<wire x1="-14.605" y1="33.655" x2="-14.605" y2="34.29" width="0.4064" layer="1"/>
 </signal>
 <signal name="+1V8/1">
