File: 7_MBUS/7_MBUS.brd (EAGLE design)
At the start: 67.4 x 44.8 mm, 23 parts, among them T1 BCP51-16, T2 BC847, T3 BC847, X1 AKL18X-02W, X12 ALLSERIALD

Commit message: change diodes
Parts:
- added R12: 39k, rcl:R0805
- added R13: 22, rcl:R0805
- added R14: 2k2, rcl:R0805
- added U$1: (no value), Mentor:1271.1000
- moved R10 168.1 mm to (15.2, 26.7), turned to 180 degrees
- moved R9 159.6 mm to (15.2, 22.9)
- moved R11 159.0 mm to (21.6, 5.08), turned to 270 degrees
- moved T3 147.8 mm to (22.9, 10.2)
- moved R8 141.6 mm to (7.62, 21.6), turned to 270 degrees
- moved R6 127.9 mm to (0.00, 31.8)
- moved R7 125.8 mm to (5.08, 10.2), turned to 180 degrees
- moved T2 125.6 mm to (6.35, 16.5), turned to 180 degrees
- moved C4 86.2 mm to (-19.7, 18.4), turned to 180 degrees
- moved R4 79.1 mm to (-14.0, 14.0), turned to 270 degrees
- moved R3 72.3 mm to (-16.5, 14.0), turned to 90 degrees
- moved D1 63.6 mm to (-24.1, 22.9), turned to 90 degrees
- moved L1 63.1 mm to (-14.0, 30.5)
- moved C3 62.5 mm to (-24.1, 14.0), turned to 90 degrees
- moved R2 58.9 mm to (-9.53, 22.9)
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Connections:
- new net N$100: R5.2, R9.2, X1.P$1
- new net N$11: R13.1
- new net N$14: R14.2, T3.3
- net 36V: now also R13.2; no longer R5.2, R9.2, X1.P$1
- net GND: now also R12.1; no longer R6.1
- net N$12: now also R14.1; no longer T3.3
Routing:
- net N$100: track 0.00 -> 28.2 mm
- net N$12: track 0.00 -> 23.5 mm
- net +12V: track 0.00 -> 21.8 mm
- net N$2: track 0.00 -> 19.5 mm
- net N$1: track 0.00 -> 18.9 mm
- net +5V: track 0.00 -> 17.1 mm
- net N$8: track 0.00 -> 16.4 mm
- net 36V: track 0.00 -> 12.2 mm
- net N$9: track 0.00 -> 12.0 mm
- net N$7: track 0.00 -> 10.7 mm
- net N$6: track 0.00 -> 8.67 mm
- net N$10: track 0.00 -> 3.16 mm
- net N$13: track 0.00 -> 3.16 mm
- net N$3: track 0.00 -> 2.28 mm
- net N$11: track 0.00 -> 1.28 mm

Commit message: use new lib
Parts:
- removed X12: ALLSERIALD, AllSerial:DAUGHTER-THT
- added X2: ALLSERIALSLAVE, AllSerialv2:DAUGHTER-THT
Connections:
- net +12V: now also X2.19; no longer X12.20
- net +5V: now also X2.18, X2.20; no longer X12.18, X12.7
- net GND: now also X2.1; no longer X12.19
- net N$8: now also X2.17; no longer X12.5
- net N$9: now also X2.8; no longer X12.8
Routing:
- net +5V: track 17.1 -> 2.04 mm
- net N$9: track 12.0 -> 10.2 mm
- net N$8: track 16.4 -> 14.6 mm
- net +12V: track 21.8 -> 20.0 mm
Changed lines of the file:
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@@
 <?xml version="1.0" encoding="utf-8"?>
 <!DOCTYPE eagle SYSTEM "eagle.dtd">
-<eagle version="7.7.0">
+<eagle version="7.6.0">
 <drawing>
 <settings>
@@
 </autorouter>
 <elements>
-<element name="X12" library="AllSerial" package="DAUGHTER-THT" value="ALLSERIALD" x="0" y="0"/>
 <element name="U1" library="microbuilder" package="SOIC8_150MIL" value="" x="-13.97" y="19.05" rot="R270"/>
 <element name="C1" library="rcl" package="C0805" value="100n" x="-6.35" y="17.145"/>
@@
 <element name="U$1" library="Mentor" package="1271.1000" value="" x="-2.54" y="34.29"/>
 <element name="R14" library="rcl" package="R0805" value="2k2" x="-33.02" y="-8.89"/>
+<element name="X2" library="AllSerialv2" package="DAUGHTER-THT" value="ALLSERIALSLAVE" x="0" y="0"/>
 </elements>
 <signals>
 <signal name="GND" airwireshidden="yes">
-<contactref element="X12" pad="19"/>
 <polygon width="0.254" layer="16">
 <vertex x="-34.29" y="44.45"/>
@@
 <contactref element="R10" pad="1"/>
 <contactref element="R12" pad="1"/>
+<contactref element="X2" pad="1"/>
 <wire x1="5.4" y1="17.61" x2="16.19" y2="26.67" width="0" layer="19" extent="1-1"/>
 <wire x1="-2.68" y1="12.7" x2="5.4" y2="17.61" width="0" layer="19" extent="1-1"/>
@@
 <wire x1="-20.635" y1="18.415" x2="-16.57" y2="17.145" width="0" layer="19" extent="1-1"/>
 <wire x1="-24.13" y1="11.57" x2="-20.635" y2="18.415" width="0" layer="19" extent="1-1"/>
-<wire x1="-11.43" y1="6.985" x2="-13.97" y2="14.92" width="0" layer="19" extent="1-1"/>
+<wire x1="-11.43" y1="4.445" x2="-13.97" y2="14.92" width="0" layer="19" extent="1-1"/>
 <wire x1="23.81" y1="9.06" x2="16.19" y2="26.67" width="0" layer="19" extent="1-1"/>
 <wire x1="1.27" y1="42.86" x2="16.19" y2="26.67" width="0" layer="19" extent="1-1"/>
@@
 </signal>
 <signal name="+12V">
-<contactref element="X12" pad="20"/>
 <contactref element="U1" pad="6"/>
 <contactref element="C2" pad="+"/>
@@
 <wire x1="-7.3" y1="17.145" x2="-7.3" y2="18.1" width="0.8128" layer="1"/>
 <wire x1="-7.3" y1="18.1" x2="-6.67" y2="18.73" width="0.8128" layer="1"/>
-<wire x1="-11.43" y1="4.445" x2="-10.16" y2="5.715" width="0.4064" layer="1"/>
 <wire x1="-10.16" y1="5.715" x2="-10.16" y2="8.89" width="0.4064" layer="1"/>
 <wire x1="-7.48" y1="12.7" x2="-7.48" y2="11.57" width="0.4064" layer="1"/>
 <wire x1="-7.48" y1="11.57" x2="-10.16" y2="8.89" width="0.4064" layer="1"/>
+<contactref element="X2" pad="19"/>
+<wire x1="-8.89" y1="6.985" x2="-10.16" y2="5.715" width="0" layer="19" extent="1-1"/>
 </signal>
 <signal name="+5V">
-<contactref element="X12" pad="18"/>
-<contactref element="X12" pad="7"/>
 <contactref element="R7" pad="2"/>
-<wire x1="-8.89" y1="4.445" x2="-7.62" y2="5.715" width="0.6096" layer="1"/>
-<wire x1="-7.62" y1="5.715" x2="2.54" y2="5.715" width="0.6096" layer="1"/>
-<wire x1="2.54" y1="5.715" x2="3.81" y2="6.985" width="0.6096" layer="1"/>
-<wire x1="3.81" y1="6.985" x2="3.81" y2="8.255" width="0.4064" layer="1"/>
 <wire x1="4.13" y1="10.16" x2="4.13" y2="8.575" width="0.4064" layer="1"/>
 <wire x1="4.13" y1="8.575" x2="3.81" y2="8.255" width="0.4064" layer="1"/>
+<contactref element="X2" pad="20"/>
+<contactref element="X2" pad="18"/>
+<wire x1="-6.35" y1="6.985" x2="3.81" y2="8.255" width="0" layer="19" extent="1-1"/>
+<wire x1="-11.43" y1="6.985" x2="-6.35" y2="6.985" width="0" layer="19" extent="1-1"/>
 </signal>
 <signal name="N$2">
@@
 <contactref element="T2" pad="3"/>
 <contactref element="R7" pad="1"/>
-<contactref element="X12" pad="8"/>
-<wire x1="3.81" y1="4.445" x2="5.08" y2="5.715" width="0.4064" layer="1"/>
 <wire x1="5.08" y1="5.715" x2="5.08" y2="7.62" width="0.4064" layer="1"/>
 <wire x1="5.08" y1="7.62" x2="6.03" y2="8.57" width="0.4064" layer="1"/>
@@
 <wire x1="6.03" y1="10.16" x2="6.03" y2="12.38" width="0.4064" layer="1"/>
 <wire x1="6.03" y1="12.38" x2="6.35" y2="12.7" width="0.4064" layer="1"/>
+<contactref element="X2" pad="8"/>
+<wire x1="6.35" y1="4.445" x2="5.08" y2="5.715" width="0" layer="19" extent="1-1"/>
 </signal>
 <signal name="N$10">
@@
 </signal>
 <signal name="N$8">
-<contactref element="X12" pad="5"/>
 <contactref element="R11" pad="2"/>
-<wire x1="6.35" y1="6.985" x2="7.62" y2="5.715" width="0.4064" layer="1"/>
 <wire x1="7.62" y1="5.715" x2="17.145" y2="5.715" width="0.4064" layer="1"/>
 <wire x1="21.59" y1="4.13" x2="18.73" y2="4.13" width="0.4064" layer="1"/>
 <wire x1="18.73" y1="4.13" x2="17.145" y2="5.715" width="0.4064" layer="1"/>
+<contactref element="X2" pad="17"/>
+<wire x1="-3.81" y1="6.985" x2="7.62" y2="5.715" width="0" layer="19" extent="1-1"/>
 </signal>
 <signal name="N$100">
