File: Mainboards/WiFi ESP32/Board S2/WiFiMaster.kicad_sch (KiCad schematic)
At the start: 63 parts, among them IC1 MCP170X, IC2 NCP1117ST, IC3 ADuM142E1BRZ, IC4 ADuM142E1BRZ, IC5 ADuM142E1BRZ, IC6 IL0505, IC7 NCP1117ST, IC8 TPS61041, J1 USB_C_Receptacle_USB2.0, J2 Conn_02x05_Odd_Even, U1 ESP32-S3-MINI-1, X1 AKL18X-04W, X2 ALLSERIALMASTERM

Commit message: Improve libraries
Parts:
- renumbered C5 to C1, R8 to R12, R10 to R13
Changed lines of the file:
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@@
 (kicad_sch
-	(version 20231120)
+	(version 20250114)
 	(generator "eeschema")
-	(generator_version "8.0")
+	(generator_version "9.0")
 	(paper "A4")
 	(title_block
@@
 	(label "DTR_B"
 		(at 194.31 39.37 180)
-		(fields_autoplaced yes)
 		(effects
 			(font
@@
 	(label "DCD_A"
 		(at 138.43 161.29 180)
-		(fields_autoplaced yes)
 		(effects
 			(font
@@
 	(label "DSR_A"
 		(at 104.14 54.61 0)
-		(fields_autoplaced yes)
 		(effects
 			(font
@@
 	(label "GP_A"
 		(at 138.43 48.26 180)
-		(fields_autoplaced yes)
 		(effects
 			(font
@@
 	(label "TXEN_A"
 		(at 102.87 139.7 0)
-		(fields_autoplaced yes)
 		(effects
 			(font
@@
 	(label "DSR_B"
 		(at 171.45 54.61 0)
-		(fields_autoplaced yes)
 		(effects
 			(font
@@
 	(label "RST"
 		(at 138.43 147.32 180)
-		(fields_autoplaced yes)
 		(effects
 			(font
@@
 	(label "RTS_B"
 		(at 171.45 41.91 0)
-		(fields_autoplaced yes)
 		(effects
 			(font
@@
 	(label "LED3"
 		(at 39.37 166.37 90)
-		(fields_autoplaced yes)
 		(effects
 			(font
@@
 	(label "RTS_A"
 		(at 104.14 57.15 0)
-		(fields_autoplaced yes)
 		(effects
 			(font
@@
 	(label "LED2"
 		(at 64.77 172.72 180)
-		(fields_autoplaced yes)
 		(effects
 			(font
@@
 	(label "CTS_A"
 		(at 60.96 119.38 180)
-		(fields_autoplaced yes)
 		(effects
 			(font
@@
 	(label "DTR_A"
 		(at 102.87 137.16 0)
-		(fields_autoplaced yes)
 		(effects
 			(font
@@
 	(label "TXD_A"
 		(at 78.74 64.77 180)
-		(fields_autoplaced yes)
 		(effects
 			(font
@@
 	(label "TXD_A"
 		(at 138.43 140.97 180)
-		(fields_autoplaced yes)
 		(effects
 			(font
@@
 	(label "RXD_A"
 		(at 102.87 114.3 0)
-		(fields_autoplaced yes)
 		(effects
 			(font
@@
 	(label "RST_B"
 		(at 194.31 57.15 180)
-		(fields_autoplaced yes)
 		(effects
 			(font
@@
 	(label "CTS_A"
 		(at 104.14 62.23 0)
-		(fields_autoplaced yes)
 		(effects
 			(font
@@
 	(label "DSR_A"
 		(at 102.87 132.08 0)
-		(fields_autoplaced yes)
 		(effects
 			(font
@@
 	(label "RTS_B"
 		(at 194.31 34.29 180)
-		(fields_autoplaced yes)
 		(effects
 			(font
@@
 	(label "DSR_A"
 		(at 138.43 54.61 180)
-		(fields_autoplaced yes)
 		(effects
 			(font
@@
 	(label "RI_A"
 		(at 102.87 129.54 0)
-		(fields_autoplaced yes)
 		(effects
 			(font
@@
 	(label "RXD_B"
 		(at 171.45 104.14 0)
-		(fields_autoplaced yes)
 		(effects
 			(font
@@
 	(label "LED3"
 		(at 64.77 170.18 180)
-		(fields_autoplaced yes)
 		(effects
 			(font
@@
 	(label "GP_A"
 		(at 102.87 134.62 0)
-		(fields_autoplaced yes)
 		(effects
 			(font
@@
 	(label "TXEN_A"
 		(at 78.74 59.69 180)
-		(fields_autoplaced yes)
 		(effects
 			(font
@@
 	(label "RI_A"
 		(at 78.74 54.61 180)
-		(fields_autoplaced yes)
 		(effects
 			(font
@@
 	(label "TXD_A"
 		(at 102.87 111.76 0)
-		(fields_autoplaced yes)
 		(effects
 			(font
@@
 	(label "TXEN_A"
 		(at 138.43 91.44 180)
-		(fields_autoplaced yes)
 		(effects
 			(font
@@
 	(label "GP_B"
 		(at 194.31 54.61 180)
-		(fields_autoplaced yes)
 		(effects
 			(font
@@
 	(label "DTR_A"
 		(at 104.14 59.69 0)
-		(fields_autoplaced yes)
 		(effects
 			(font
@@
 	(label "TXD_B"
 		(at 171.45 140.97 0)
-		(fields_autoplaced yes)
 		(effects
 			(font
@@
 	(label "USB_D-"
 		(at 54.61 43.18 0)
-		(fields_autoplaced yes)
 		(effects
 			(font
@@
 	(label "RI_B"
 		(at 171.45 60.96 0)
-		(fields_autoplaced yes)
 		(effects
 			(font
@@
 	(label "BTN"
 		(at 36.83 111.76 180)
-		(fields_autoplaced yes)
 		(effects
 			(font
@@
 	(label "RST_B"
 		(at 171.45 147.32 0)
-		(fields_autoplaced yes)
 		(effects
 			(font
@@
 	(label "RI_A"
 		(at 138.43 60.96 180)
-		(fields_autoplaced yes)
 		(effects
 			(font
@@
 	(label "USB_D+"
 		(at 54.61 40.64 0)
-		(fields_autoplaced yes)
 		(effects
 			(font
@@
 	(label "RTS_A"
 		(at 60.96 116.84 180)
-		(fields_autoplaced yes)
 		(effects
 			(font
@@
 	(label "DSR_B"
 		(at 194.31 41.91 180)
-		(fields_autoplaced yes)
 		(effects
 			(font
@@
 	(label "LED1"
 		(at 64.77 175.26 180)
-		(fields_autoplaced yes)
 		(effects
 			(font
@@
 	(label "RI_B"
 		(at 194.31 46.99 180)
-		(fields_autoplaced yes)
 		(effects
 			(font
@@
 	(label "RXD_A"
 		(at 78.74 57.15 180)
-		(fields_autoplaced yes)
 		(effects
 			(font
@@
 	(label "LED4"
 		(at 102.87 170.18 0)
-		(fields_autoplaced yes)
 		(effects
 			(font
@@
 	(label "LED2"
 		(at 30.48 166.37 90)
-		(fields_autoplaced yes)
 		(effects
 			(font
@@
 	(label "LED4"
 		(at 48.26 166.37 90)
-		(fields_autoplaced yes)
 		(effects
 			(font
@@
 	(label "CTS_B"
 		(at 194.31 36.83 180)
-		(fields_autoplaced yes)
 		(effects
 			(font
@@
 	(label "TXEN_B"
 		(at 194.31 52.07 180)
-		(fields_autoplaced yes)
 		(effects
 			(font
@@
 	(label "GP_B"
 		(at 171.45 48.26 0)
-		(fields_autoplaced yes)
 		(effects
 			(font
@@
 	(label "DCD_B"
 		(at 194.31 44.45 180)
-		(fields_autoplaced yes)
 		(effects
 			(font
@@
 	(label "BTN"
 		(at 102.87 172.72 0)
-		(fields_autoplaced yes)
 		(effects
 			(font
@@
 	(label "GND"
 		(at 25.4 82.55 180)
-		(fields_autoplaced yes)
 		(effects
 			(font
@@
 	(label "CTS_A"
 		(at 138.43 153.67 180)
-		(fields_autoplaced yes)
 		(effects
 			(font
@@
 	(label "TXEN_B"
 		(at 171.45 91.44 0)
-		(fields_autoplaced yes)
 		(effects
 			(font
@@
 	(label "RTS_A"
 		(at 138.43 41.91 180)
-		(fields_autoplaced yes)
 		(effects
 			(font
@@
 	(label "SHLD"
 		(at 19.05 72.39 0)
-		(fields_autoplaced yes)
 		(effects
 			(font
@@
 	(label "USB_D-"
 		(at 102.87 121.92 0)
-		(fields_autoplaced yes)
 		(effects
 			(font
@@
 	(label "RXD_B"
 		(at 194.31 31.75 180)
-		(fields_autoplaced yes)
 		(effects
 			(font
@@
 	(label "DCD_A"
 		(at 102.87 142.24 0)
-		(fields_autoplaced yes)
 		(effects
 			(font
@@
 	(label "DTR_B"
 		(at 171.45 97.79 0)
-		(fields_autoplaced yes)
 		(effects
 			(font
@@
 	(label "USB_D+"
 		(at 102.87 119.38 0)
-		(fields_autoplaced yes)
 		(effects
 			(font
@@
 	(label "LED1"
 		(at 21.59 166.37 90)
-		(fields_autoplaced yes)
 		(effects
 			(font
@@
 	(label "CTS_B"
 		(at 171.45 153.67 0)
-		(fields_autoplaced yes)
 		(effects
 			(font
@@
 	(label "DCD_A"
 		(at 78.74 62.23 180)
-		(fields_autoplaced yes)
 		(effects
 			(font
@@
 	(label "DCD_B"
 		(at 171.45 161.29 0)
-		(fields_autoplaced yes)
 		(effects
 			(font
@@
 	(label "RXD_A"
 		(at 138.43 104.14 180)
-		(fields_autoplaced yes)
 		(effects
 			(font
@@
 	(label "DTR_A"
 		(at 138.43 97.79 180)
-		(fields_autoplaced yes)
 		(effects
 			(font
@@
 	(label "TXD_B"
 		(at 194.31 29.21 180)
-		(fields_autoplaced yes)
 		(effects
 			(font
@@
 		(on_board yes)
 		(dnp no)
-		(property "Reference" "R8"
+		(property "Reference" "R12"
 			(at 38.1 102.87 0)
 			(effects
@@
 		(on_board yes)
 		(dnp no)
-		(property "Reference" "#PWR015"
+		(property "Reference" "#PWR036"
 			(at 39.37 130.81 0)
 			(effects
@@
 		(on_board yes)
 		(dnp no)
-		(property "Reference" "R10"
+		(property "Reference" "R13"
 			(at 55.88 102.87 0)
 			(effects
@@
 		(on_board yes)
 		(dnp no)
-		(property "Reference" "#PWR018"
+		(property "Reference" "#PWR037"
 			(at 49.53 104.14 0)
 			(effects
@@
 		(on_board yes)
 		(dnp no)
-		(property "Reference" "#PWR014"
+		(property "Reference" "#PWR035"
 			(at 39.37 104.14 0)
 			(effects
@@
 		(on_board yes)
 		(dnp no)
-		(property "Reference" "C5"
+		(property "Reference" "C1"
 			(at 45.72 115.57 90)
 			(effects
@@
 		(on_board yes)
 		(dnp no)
-		(property "Reference" "#PWR019"
+		(property "Reference" "#PWR038"
 			(at 57.15 104.14 0)
 			(effects
@@
 		)
 	)
+	(embedded_fonts no)
 )
