File: Slaveboards/eBus/Board/AllSerial eBus.kicad_sch (KiCad schematic)
At the start: 40 parts, among them J3 Conn_01x02, Q1 Q_PNP_BCEC, Q2 BC847, Q3 BC857, Q4 BC847, Q5 Q_PNP_BCEC, Q6 BC847, U1 LM293, X1 AllSerial_Connector

Commit message: Improve libraries
Parts:
- D7: footprint LED_SMD:LED_0805_2012Metric -> LED_SMD:LED_0603_1608Metric
Changed lines of the file:
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@@
 			)
 		)
-		(property "Footprint" "LED_SMD:LED_0805_2012Metric"
+		(property "Footprint" "LED_SMD:LED_0603_1608Metric"
 			(at 189.23 41.91 0)
 			(effects
